File: stm32f0can.kicad_pcb (KiCad board)
At the start: 4 copper layers, 63.5 x 38.1 mm, 34 parts, among them J1 Screw_Terminal_01x02, J2 Conn_01x04_Female, J3 Conn_02x05_Odd_Even, J4 Conn_01x04_Female, J5 Conn_01x04_Female, J6 Conn_01x03_Female, J7 Conn_01x04_Female, J8 Conn_01x04_Female, U2 IFX1050GVIO

Commit message: added git repo on silklayer
Other:
- board text added: "https://github.com/COLVERTYETY/stm32canProto"
Changed lines of the file:
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@@
   (general
     (thickness 1.6)
-    (drawings 47)
+    (drawings 48)
     (tracks 217)
     (zones 0)
@@
       (net 31 can_tx))
   )
+  (gr_text https://github.com/COLVERTYETY/stm32canProto (at 130.937 126.8476) (layer B.SilkS)
+    (effects (font (size 1 1) (thickness 0.15)) (justify mirror))
+  )
   (gr_text "active low" (at 105.8926 118.3132 -90) (layer F.SilkS)

Commit message: drc
Other:
- board text added: "."
Changed lines of the file:
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@@
   (general
     (thickness 1.6)
-    (drawings 48)
-    (tracks 217)
+    (drawings 49)
+    (tracks 219)
     (zones 0)
     (modules 34)
@@
       (net 31 can_tx))
   )
+  (gr_text . (at 116.1034 113.0808) (layer F.SilkS)
+    (effects (font (size 1 1) (thickness 0.15)))
+  )
   (gr_text https://github.com/COLVERTYETY/stm32canProto (at 130.937 126.8476) (layer B.SilkS)
     (effects (font (size 1 1) (thickness 0.15)) (justify mirror))
@@
   (segment (start 141.7701 113.03) (end 141.8336 113.0935) (width 0.25) (layer F.Cu) (net 1))
   (segment (start 139.7 113.03) (end 141.7701 113.03) (width 0.5) (layer F.Cu) (net 1))
-  (segment (start 124.635003 116.930001) (end 125.690799 116.930001) (width 0.4) (layer F.Cu) (net 1))
-  (segment (start 124.485002 116.78) (end 124.635003 116.930001) (width 0.4) (layer F.Cu) (net 1))
-  (segment (start 123.6 116.78) (end 124.485002 116.78) (width 0.4) (layer F.Cu) (net 1))
-  (segment (start 125.690799 116.930001) (end 125.9713 116.6495) (width 0.4) (layer F.Cu) (net 1))
   (via (at 125.996837 116.662644) (size 0.8) (drill 0.4) (layers F.Cu B.Cu) (net 1))
   (segment (start 125.983693 116.6495) (end 125.996837 116.662644) (width 0.25) (layer F.Cu) (net 1))
@@
   (segment (start 137.254999 100.235001) (end 134.525001 100.235001) (width 0.25) (layer In1.Cu) (net 1))
   (segment (start 138.43 99.06) (end 137.254999 100.235001) (width 0.25) (layer In1.Cu) (net 1))
+  (segment (start 125.996837 116.662644) (end 125.958156 116.662644) (width 0.25) (layer F.Cu) (net 1))
+  (segment (start 125.723058 116.662644) (end 125.996837 116.662644) (width 0.25) (layer F.Cu) (net 1))
+  (segment (start 125.455701 116.930001) (end 125.723058 116.662644) (width 0.25) (layer F.Cu) (net 1))
+  (segment (start 124.609698 116.78) (end 124.759699 116.930001) (width 0.25) (layer F.Cu) (net 1))
+  (segment (start 124.759699 116.930001) (end 125.455701 116.930001) (width 0.25) (layer F.Cu) (net 1))
+  (segment (start 123.6 116.78) (end 124.609698 116.78) (width 0.25) (layer F.Cu) (net 1))
   (segment (start 127.715 112.99) (end 128.27 112.99) (width 0.25) (layer F.Cu) (net 2))
   (segment (start 119.38 105.19) (end 119.6 105.41) (width 0.25) (layer F.Cu) (net 2))
@@
   (segment (start 145.81 113.03) (end 147.32 111.52) (width 0.8) (layer F.Cu) (net 14))
   (segment (start 144.61 113.03) (end 145.81 113.03) (width 0.8) (layer F.Cu) (net 14))
-  (segment (start 147.32 102.87) (end 149.86 100.33) (width 1) (layer F.Cu) (net 14))
   (segment (start 147.32 111.52) (end 147.32 102.87) (width 1) (layer F.Cu) (net 14))
   (segment (start 149.86 100.33) (end 157.48 100.33) (width 1) (layer F.Cu) (net 14))
+  (segment (start 147.32 102.87) (end 149.86 100.33) (width 1) (layer F.Cu) (net 14))
   (segment (start 144.61 114.3) (end 146.05 114.3) (width 0.8) (layer F.Cu) (net 15))
   (segment (start 149.86 110.49) (end 149.86 105.41) (width 1) (layer F.Cu) (net 15))
